File: mobo/mobo.kicad_pcb (KiCad board)
At the start: 2 copper layers, 100 x 100 mm, 5 parts, among them U1 Z-turn

Commit message: 5V Power supply schematic + place
Parts:
- added C1: 22nF, Capacitors_SMD:C_0805_HandSoldering, F.Cu at (98.5, 54.5)
- added C2: 82pF, Capacitors_SMD:C_0805_HandSoldering, F.Cu at (100.0, 64.8)
- added C3: 22nF, Capacitors_SMD:C_0805_HandSoldering, F.Cu at (98.5, 49.5)
- added C4: 22nF, Capacitors_SMD:C_0805_HandSoldering, F.Cu at (96.0, 49.5)
- added C5: 2.2nF, Capacitors_SMD:C_0805_HandSoldering, F.Cu at (105.5, 59.8)
- added L1: 4.7uH, Inductors:Inductor_Taiyo-Yuden_MD-5050, F.Cu at (104.2, 47.5)
- added R1: 24.9k, Resistors_SMD:R_0805_HandSoldering, F.Cu at (100.0, 62.2)
- added R2: 4.75k, Resistors_SMD:R_0805_HandSoldering, F.Cu at (100.0, 59.8)
- added R3: 8.25k, Resistors_SMD:R_0805_HandSoldering, F.Cu at (105.5, 62.2)
- added U2: ncp3170, Housings_SOIC:SOIC-8_3.9x4.9mm_Pitch1.27mm, F.Cu at (104.8, 55.0)
Connections:
- net GND renamed GNDD
- U1 pad 1: Net-(U1-Pad1) -> +5VD
- U1 pad 81: Net-(U1-Pad81) -> +5VD

Commit message: started h-bridge
Parts:
- added C7: 100nF, Capacitors_SMD:C_0805_HandSoldering, F.Cu at (112.0, 121.5)
- added C9: 100nF, Capacitors_SMD:C_0805_HandSoldering, F.Cu at (98.5, 120.8)
- added U3: TLE5206-2G, Infineon:PG-TO263-7-1, F.Cu at (100.0, 127.0)
- added U4: TLE5206-2G, Infineon:PG-TO263-7-1, F.Cu at (113.5, 127.0)
Connections:
- U1 pad 3: Net-(U1-Pad3) -> +3V3
- U1 pad 83: Net-(U1-Pad83) -> +3V3
